File: KiCAD/ROV CTD.kicad_pcb (KiCad board)
At the start: 2 copper layers, 73.7 x 23.4 mm, 35 parts, among them J10 1Wire1, J11 1Wire2, J12 1Wire3, J4 Bottom - Middle, J6 Main In, J7 Bottom - Middle, J8 Middle - Top, J9 Middle - Top, U2 ATtiny1614-Arduino, U3 AP63205WU, U6 MAX3072E

Commit message: .
Parts:
- moved J8 1.40 mm to (139.4, 66.7)
- moved J9 0.13 mm to (139.4, 66.7)
Changed lines of the file:
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@@
 	(footprint "Connector_PinSocket_1.27mm:PinSocket_2x03_P1.27mm_Vertical_SMD"
 		(layer "F.Cu")
-		(at 139.446 68.072 180)
+		(at 139.446 66.675 180)
 		(descr "surface-mounted straight socket strip, 2x03, 1.27mm pitch, double rows (from Kicad 4.0.7!), script generated")
 		(tags "Surface mounted socket strip SMD 2x03 1.27mm double row")
@@
 	(footprint "Connector_PinHeader_1.27mm:PinHeader_2x03_P1.27mm_Vertical_SMD"
 		(layer "B.Cu")
-		(at 139.446 66.802)
+		(at 139.446 66.675)
 		(descr "surface-mounted straight pin header, 2x03, 1.27mm pitch, double rows")
 		(tags "Surface mounted pin header SMD 2x03 1.27mm double row")
@@
 	)
 	(segment
+		(start 172.9955 82.804)
+		(end 172.9955 78.74)
+		(width 0.7)
+		(layer "B.Cu")
+		(net "+5V_Mid")
+	)
+	(segment
+		(start 172.9955 77.4915)
+		(end 168.656 73.152)
+		(width 0.7)
+		(layer "B.Cu")
+		(net "+5V_Mid")
+	)
+	(segment
+		(start 165.735 84.57)
+		(end 166.326 83.979)
+		(width 0.7)
+		(layer "B.Cu")
+		(net "+5V_Mid")
+	)
+	(segment
+		(start 164.465 85.77)
+		(end 165.735 85.77)
+		(width 0.7)
+		(layer "B.Cu")
+		(net "+5V_Mid")
+	)
+	(segment
+		(start 171.8205 83.979)
+		(end 172.9955 82.804)
+		(width 0.7)
+		(layer "B.Cu")
+		(net "+5V_Mid")
+	)
+	(segment
+		(start 172.9955 78.74)
+		(end 172.9955 77.4915)
+		(width 0.7)
+		(layer "B.Cu")
+		(net "+5V_Mid")
+	)
+	(segment
+		(start 166.326 83.979)
+		(end 171.8205 83.979)
+		(width 0.7)
+		(layer "B.Cu")
+		(net "+5V_Mid")
+	)
+	(segment
+		(start 161.544 73.152)
+		(end 168.656 73.152)
+		(width 0.7)
+		(layer "B.Cu")
+		(net "+5V_Mid")
+	)
+	(segment
+		(start 165.735 85.77)
+		(end 165.735 84.57)
+		(width 0.7)
+		(layer "B.Cu")
+		(net "+5V_Mid")
+	)
+	(segment
 		(start 168.656 75.692)
 		(end 165.1 75.692)
@@
 		(net "/NeoPixle")
 	)
-	(segment
-		(start 172.9955 82.804)
-		(end 172.9955 78.74)
-		(width 0.7)
-		(layer "B.Cu")
-		(net "+5V_Mid")
-	)
-	(segment
-		(start 172.9955 77.4915)
-		(end 168.656 73.152)
-		(width 0.7)
-		(layer "B.Cu")
-		(net "+5V_Mid")
-	)
-	(segment
-		(start 165.735 84.57)
-		(end 166.326 83.979)
-		(width 0.7)
-		(layer "B.Cu")
-		(net "+5V_Mid")
-	)
-	(segment
-		(start 164.465 85.77)
-		(end 165.735 85.77)
-		(width 0.7)
-		(layer "B.Cu")
-		(net "+5V_Mid")
-	)
-	(segment
-		(start 171.8205 83.979)
-		(end 172.9955 82.804)
-		(width 0.7)
-		(layer "B.Cu")
-		(net "+5V_Mid")
-	)
-	(segment
-		(start 172.9955 78.74)
-		(end 172.9955 77.4915)
-		(width 0.7)
-		(layer "B.Cu")
-		(net "+5V_Mid")
-	)
-	(segment
-		(start 166.326 83.979)
-		(end 171.8205 83.979)
-		(width 0.7)
-		(layer "B.Cu")
-		(net "+5V_Mid")
-	)
-	(segment
-		(start 161.544 73.152)
-		(end 168.656 73.152)
-		(width 0.7)
-		(layer "B.Cu")
-		(net "+5V_Mid")
-	)
-	(segment
-		(start 165.735 85.77)
-		(end 165.735 84.57)
-		(width 0.7)
-		(layer "B.Cu")
-		(net "+5V_Mid")
-	)
 	(via
 		(at 184.785 70.58175)
@@
 	)
 	(segment
-		(start 167.005 85.77)
-		(end 168.275 85.77)
-		(width 0.7)
-		(layer "B.Cu")
-		(net "V_in_Mid")
-	)
-	(segment
 		(start 141.396 68.072)
 		(end 141.732 68.072)
@@
 		(net "unconnected-(J9-Pin_4-Pad4)")
 	)
+	(segment
+		(start 167.005 85.77)
+		(end 168.275 85.77)
+		(width 0.7)
+		(layer "B.Cu")
+		(net "V_in_Mid")
+	)
 	(zone
