File: KiCAD/ROV CTD.kicad_pcb (KiCad board)
At the start: 2 copper layers, 73.7 x 23.4 mm, 55 parts, among them J4 Bottom - Middle, J6 Main In, J7 Bottom - Middle, J8 Middle - Top, J9 Middle - Top, U1 AL8805W5, U2 ATtiny1614-Arduino, U3 AP63205WU, U6 MAX3072E

Commit message: cleanup
Parts:
- removed C10, C11, C12, C18: 47uF, Capacitor_SMD:C_0805_2012Metric_Pad1.18x1.45mm_HandSolder
- removed C2: 2.2uF, Capacitor_SMD:C_0805_2012Metric_Pad1.18x1.45mm_HandSolder
- removed C5: 1uF, Capacitor_SMD:C_0805_2012Metric_Pad1.18x1.45mm_HandSolder
- removed C8: 100nF, Capacitor_SMD:C_0805_2012Metric_Pad1.18x1.45mm_HandSolder
- removed D1: CXA1304, KiCad Footprints:LED - CXA1304
- removed D11: Status, LED_SMD:LED_0805_2012Metric_Pad1.15x1.40mm_HandSolder
- removed D2: BAT54S, Package_TO_SOT_SMD:SOT-23
- removed D6, D7, D8, D9: Inolux_IN-PI554FCH, LED_SMD:LED_Inolux_IN-PI554FCH_PLCC4_5.0x5.0mm_P3.2mm
- removed J9: Middle - Top, Connector_PinHeader_1.27mm:PinHeader_2x03_P1.27mm_Vertical_SMD
- removed L1: SRN6045-330M, KiCad Footprints:inductor_33uH
- removed R1, R2, R5, R6: 0.5, Resistor_SMD:R_1206_3216Metric_Pad1.30x1.75mm_HandSolder
- removed R12, R13: 330, Resistor_SMD:R_0805_2012Metric_Pad1.20x1.40mm_HandSolder
- removed R14: 1k, Resistor_SMD:R_0805_2012Metric_Pad1.20x1.40mm_HandSolder
- removed R3, R8: 10k, Resistor_SMD:R_0805_2012Metric_Pad1.20x1.40mm_HandSolder
- removed TH1: NTCG203NH103JTDS, Resistor_SMD:R_0805_2012Metric_Pad1.20x1.40mm_HandSolder
- removed U1: AL8805W5, TO_SOT_Packages_SMD:SOT-23-5
Connections:
- J7 pad 11: /STATUS -> unconnected-(J7-Pin_11-Pad11)
- J7 pad 6: /Neo_Mid -> unconnected-(J7-Pin_6-Pad6)
- J7 pad 9: /PWM -> unconnected-(J7-Pin_9-Pad9)
- J8 pad 3: /Neo_Mid -> unconnected-(J8-Pin_3-Pad3)
- J8 pad 4: /LED-_L -> unconnected-(J8-Pin_4-Pad4)
- J8 pad 5: /STATUS -> unconnected-(J8-Pin_5-Pad5)
- J8 pad 6: /LED+_L -> unconnected-(J8-Pin_6-Pad6)
Routing:
- net /Status/Temp: track 38.0 -> 0.00 mm, vias 1 -> 0
- net V_in_Mid: track 33.2 -> 1.27 mm, vias 1 -> 0
- net /LED+_L: track 29.6 -> 0.00 mm, vias 3 -> 0
- net /Neo_Mid: track 28.3 -> 0.00 mm, vias 1 -> 0
- net /STATUS: track 28.0 -> 0.00 mm, vias 1 -> 0
- net /PWM: track 21.3 -> 0.00 mm, vias 1 -> 0
- net /LED+_U: track 19.5 -> 0.00 mm
- net +5V_Up: track 14.7 -> 0.00 mm, vias 2 -> 0
- net GND: track 34.0 -> 19.5 mm, vias 21 -> 6
- net Net-(D7-DO): track 12.6 -> 0.00 mm
- net /LED-_L: track 12.0 -> 0.00 mm
- net /LED_SW: track 10.9 -> 0.00 mm
- net Net-(D8-DO): track 10.0 -> 0.00 mm
- net Net-(D6-DO): track 10.0 -> 0.00 mm
- net Net-(U1-CTRL): track 8.80 -> 0.00 mm, vias 2 -> 0
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- removed copper zone on F.Cu, net +5V_Up
- removed copper zone on B.Cu, net /LED+_U
- removed copper zone on B.Cu, net /LED-_U
Other:
- outline, holes or cut-outs redrawn

Commit message: .
Parts:
- added C10: 47uF, Capacitor_SMD:C_0805_2012Metric_Pad1.18x1.45mm_HandSolder, B.Cu at (172.0, 80.8)
- added C5: 100nF, Capacitor_SMD:C_0805_2012Metric_Pad1.18x1.45mm_HandSolder, B.Cu at (172.0, 78.7)
- added C6: 10pF, Capacitor_SMD:C_0805_2012Metric_Pad1.18x1.45mm_HandSolder, B.Cu at (172.0, 82.8)
- added J10: 1Wire1, Connector_PinHeader_2.54mm:PinHeader_1x03_P2.54mm_Vertical, F.Cu at (161.5, 73.2)
- added J11: 1Wire2, Connector_PinHeader_2.54mm:PinHeader_1x03_P2.54mm_Vertical, F.Cu at (165.1, 73.2)
- added J12: 1Wire3, Connector_PinHeader_2.54mm:PinHeader_1x03_P2.54mm_Vertical, F.Cu at (168.7, 73.2)
- added J9: Middle - Top, Connector_PinHeader_1.27mm:PinHeader_2x03_P1.27mm_Vertical_SMD, B.Cu at (139.4, 66.8)
- moved J8 25.7 mm to (139.4, 68.1)
Connections:
- J7 pad 6: unconnected-(J7-Pin_6-Pad6) -> /1Wire
- J8 pad 1: GND -> unconnected-(J8-Pin_1-Pad1)
- J8 pad 2: +5V_Mid -> unconnected-(J8-Pin_2-Pad2)
Routing:
- net /1Wire: track 0.00 -> 18.2 mm
- net unconnected-(J9-Pin_4-Pad4): track 0.00 -> 1.35 mm
- net +5V_Mid: track 29.4 -> 29.0 mm, vias 1 -> 0

Commit message: .
Parts:
- added U1: EZO-EC, KiCad Footprints:EZO_Conductivity_Module, F.Cu at (139.7, 76.2)

Commit message: .
Parts:
- removed J4: Bottom - Middle, Connector_PinSocket_1.27mm:PinSocket_2x06_P1.27mm_Vertical_SMD
- removed J7: Bottom - Middle, Connector_PinHeader_1.27mm:PinHeader_2x06_P1.27mm_Vertical_SMD
- removed J8: Middle - Top, Connector_PinSocket_1.27mm:PinSocket_2x03_P1.27mm_Vertical_SMD
- removed J9: Middle - Top, Connector_PinHeader_1.27mm:PinHeader_2x03_P1.27mm_Vertical_SMD
- removed the REF** at (179.1, 76.2)
- removed the REF** at (165.1, 71.1)
- removed U1: EZO-EC, KiCad Footprints:EZO_Conductivity_Module
- added J1: Conn_Coaxial, Connector_Coaxial:BNC_TEConnectivity_1478204_Vertical, B.Cu at (176.5, 71.1)
- added J13: Interface, Connector_PinSocket_2.54mm:PinSocket_1x05_P2.54mm_Vertical, F.Cu at (144.8, 71.1)
- added J14: Interface, Connector_PinHeader_2.54mm:PinHeader_1x05_P2.54mm_Horizontal, B.Cu at (158.8, 71.1)
- added M1: EZO-EC, KiCad Footprints:EZO_Conductivity_Module, F.Cu at (190.5, 76.2)
- C10, C5, C6, J6, JP1, JP2: moved to F.Cu
- moved JP1 38.8 mm to (221.0, 70.5), turned to 180 degrees
- moved D10 36.5 mm to (221.0, 85.1), turned to 180 degrees
- moved U6 35.0 mm to (219.1, 75.6)
- moved R11 34.6 mm to (217.2, 85.1), turned to 0 degrees
- moved JP2 33.1 mm to (217.8, 70.5), turned to 0 degrees
- moved J6 32.4 mm to (224.8, 81.3), turned to 180 degrees
- moved C14 30.9 mm to (217.8, 84.2), turned to 90 degrees
- moved U3 27.5 mm to (214.6, 84.2), turned to -90 degrees
- moved C3 26.2 mm to (214.6, 73.7)
- moved C4 26.1 mm to (214.6, 77.5)
- moved D5 25.3 mm to (215.9, 76.8), turned to 90 degrees
- moved D4 24.9 mm to (221.0, 83.2), turned to 180 degrees
- moved R9 23.2 mm to (210.2, 73.0), turned to 180 degrees
- moved C15 21.6 mm to (212.1, 84.2), turned to 90 degrees
- moved R7 19.2 mm to (217.2, 83.2), turned to 0 degrees
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Connections:
- C10 pad 1: +5V_Mid -> +5V
- C5 pad 1: +5V_Mid -> +5V
- C6 pad 1: +5V_Mid -> +5V
- J10 pad 1: +5V_Mid -> +5V
- J11 pad 1: +5V_Mid -> +5V
- J12 pad 1: +5V_Mid -> +5V
- U2 pad 13: /NeoPixle -> /1Wire
Routing:
- net +5V_Mid: track 29.0 -> 0.00 mm
- net Net-(J1-Ext): track 0.00 -> 27.6 mm
- net /STATUS_LED: track 26.8 -> 0.00 mm
- net /LED_PWM: track 24.1 -> 0.00 mm
- net /SERIAL_RX: track 10.9 -> 33.4 mm, vias 1 -> 0
- net /1Wire: track 18.2 -> 40.0 mm
- net GND: track 19.5 -> 0.00 mm, vias 6 -> 0
- net /SERIAL_TX: track 12.8 -> 30.5 mm, vias 1 -> 0
- net /SERIAL_DIR: track 15.8 -> 1.27 mm
- net Net-(J1-In): track 0.00 -> 14.3 mm
- net /NeoPixle: track 12.3 -> 0.00 mm
- net /A9/D9: track 11.0 -> 0.00 mm
- net /Data_A: track 13.3 -> 2.83 mm, vias 1 -> 0
- net +5V: track 63.5 -> 54.4 mm, vias 4 -> 1
- net /UPDI: track 8.75 -> 0.00 mm
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Other:
- board size 73.7 x 23.4 mm -> 99.1 x 23.4 mm

Commit message: .
Parts:
- added D6: Status, LED_SMD:LED_0805_2012Metric_Pad1.15x1.40mm_HandSolder, F.Cu at (221.0, 81.3)
- added J15: Conn_01x07_Pin, Connector_PinSocket_2.54mm:PinSocket_1x07_P2.54mm_Vertical, B.Cu at (134.5, 68.5)
- added R8: 520, Resistor_SMD:R_0805_2012Metric_Pad1.20x1.40mm_HandSolder, F.Cu at (217.2, 81.3)
- added REF**: SquashedFlySilk, KiCad Footprints:SquashedFlySilk, B.Cu at (221.0, 69.2)
- moved JP2 7.43 mm to (224.8, 67.9)
- moved C3 6.25 mm to (220.3, 76.2), turned to 0 degrees
- moved C4 5.85 mm to (220.3, 78.7), turned to 0 degrees
- moved U6 3.17 mm to (219.1, 72.4), turned to 0 degrees
- moved JP1 2.62 mm to (220.3, 67.9), turned to 0 degrees
Routing:
- net +5V: track 54.4 -> 92.4 mm, vias 1 -> 3
- net /UPDI: track 0.00 -> 30.0 mm
- net /Data_A: track 2.83 -> 20.8 mm
- net /STATUS_LED: track 0.00 -> 13.2 mm
- net /SERIAL_TX: track 30.5 -> 17.8 mm
- net /SERIAL_DIR: track 1.27 -> 12.9 mm
- net /Data_B: track 2.64 -> 10.5 mm
- net /SERIAL_RX: track 33.4 -> 26.5 mm
- net /Vmeasure: track 5.94 -> 10.5 mm, vias 0 -> 1
- net /Builtin_LED: track 13.6 -> 15.6 mm
- net GND: track 0.00 -> 1.97 mm, vias 0 -> 1
- net Net-(D6-A): track 0.00 -> 1.80 mm

Commit message: .
Parts:
- added C7: 100nF, Capacitor_SMD:C_0805_2012Metric_Pad1.18x1.45mm_HandSolder, B.Cu at (142.2, 82.5)
- added JP3: RX, Jumper:SolderJumper-2_P1.3mm_Open_TrianglePad1.0x1.5mm, B.Cu at (137.2, 82.5)
- added JP4: RX, Jumper:SolderJumper-2_P1.3mm_Open_TrianglePad1.0x1.5mm, B.Cu at (140.3, 69.8)
- added M2: MS5803-14BA, KiCad Footprints:MS5803-14BA, B.Cu at (139.7, 76.2)
- added R12: 10k, Resistor_SMD:R_0805_2012Metric_Pad1.20x1.40mm_HandSolder, B.Cu at (139.7, 82.5)
- added R13: 10k, Resistor_SMD:R_0805_2012Metric_Pad1.20x1.40mm_HandSolder, B.Cu at (137.8, 69.8)
- added R14: 2k2, Resistor_SMD:R_0805_2012Metric_Pad1.20x1.40mm_HandSolder, B.Cu at (130.8, 74.9)
- added R15: 2k2, Resistor_SMD:R_0805_2012Metric_Pad1.20x1.40mm_HandSolder, B.Cu at (130.8, 77.5)
Connections:
- J13 pad 1: unconnected-(J13-Pin_1-Pad1) -> GND
- J13 pad 2: unconnected-(J13-Pin_2-Pad2) -> +3V3
- J14 pad 1: unconnected-(J14-Pin_1-Pad1) -> GND
- J14 pad 2: unconnected-(J14-Pin_2-Pad2) -> +3V3
- J15 pad 1: unconnected-(J15-Pin_1-Pad1) -> GND
- J15 pad 2: unconnected-(J15-Pin_2-Pad2) -> +3V3
- J15 pad 3: unconnected-(J15-Pin_3-Pad3) -> /SDA/SDI
- J15 pad 4: unconnected-(J15-Pin_4-Pad4) -> /SCL/SCLK
- J15 pad 5: unconnected-(J15-Pin_5-Pad5) -> /SDO
- J15 pad 6: unconnected-(J15-Pin_6-Pad6) -> /AD/CS
- J15 pad 7: unconnected-(J15-Pin_7-Pad7) -> /PS
Routing:
- net +3V3: track 0.00 -> 31.2 mm
- net /AD/CS: track 0.00 -> 16.2 mm
- net /PS: track 0.00 -> 9.00 mm

Commit message: .
Parts:
- C7, JP3, JP4, R12, R13, R14, R15: moved to F.Cu
- moved C7 12.3 mm to (139.7, 70.5), turned to 180 degrees
- moved R13 9.44 mm to (131.4, 76.8), turned to 0 degrees
- moved R12 9.09 mm to (131.4, 78.7), turned to 0 degrees
- moved JP3 6.75 mm to (141.6, 77.5), turned to 180 degrees
- moved JP4 5.24 mm to (141.6, 74.9), turned to 180 degrees
- moved R15 2.62 mm to (131.4, 74.9)
- moved R14 2.01 mm to (131.4, 73.0)
Connections:
- J13 pad 3: unconnected-(J13-Pin_3-Pad3) -> /SCL/SCLK
- J13 pad 4: unconnected-(J13-Pin_4-Pad4) -> /SDA/SDI
- J13 pad 5: unconnected-(J13-Pin_5-Pad5) -> /SDO
Routing:
- net /SDA/SDI: track 0.00 -> 20.0 mm, vias 0 -> 1
- net /SCL/SCLK: track 0.00 -> 17.1 mm, vias 0 -> 1
- net /SDO: track 0.00 -> 14.6 mm, vias 0 -> 1
- net /PS: track 9.00 -> 18.1 mm, vias 0 -> 1
- net +3V3: track 31.2 -> 34.9 mm
- net /AD/CS: track 16.2 -> 16.8 mm, vias 0 -> 1
