File: KiCAD/ROV CTD.kicad_pcb (KiCad board)
At the start: 2 copper layers, 99.1 x 23.4 mm, 45 parts, among them J1 Conn_Coaxial, J10 1Wire1, J11 1Wire2, J12 1Wire3, J13 Interface, J14 Interface, J15 Conn_01x07_Pin, J6 Main In, M1 EZO-EC, M2 MS5803-14BA, U2 ATtiny1614-Arduino, U3 AP63205WU, U6 MAX3072E

Commit message: .
Parts:
- removed D6: Status, LED_SMD:LED_0805_2012Metric_Pad1.15x1.40mm_HandSolder
- removed J10: 1Wire1, Connector_PinHeader_2.54mm:PinHeader_1x03_P2.54mm_Vertical
- removed J11: 1Wire2, Connector_PinHeader_2.54mm:PinHeader_1x03_P2.54mm_Vertical
- removed J12: 1Wire3, Connector_PinHeader_2.54mm:PinHeader_1x03_P2.54mm_Vertical
- removed R8: 520, Resistor_SMD:R_0805_2012Metric_Pad1.20x1.40mm_HandSolder
- added C8: 100nF, Capacitor_SMD:C_0805_2012Metric_Pad1.18x1.45mm_HandSolder, B.Cu at (139.7, 81.9)
- added H1: Through Hole, MountingHole:MountingHole_3mm, F.Cu at (139.7, 66.7)
- added H2: Through Hole, MountingHole:MountingHole_3mm, F.Cu at (139.7, 85.7)
- J13: value Interface -> Head Connector; footprint Connector_PinSocket_2.54mm:PinSocket_1x05_P2.54mm_Vertical -> Connector_PinSocket_2.54mm:PinSocket_1x04_P2.54mm_Vertical
- J14: value Interface -> Head Connector; footprint Connector_PinHeader_2.54mm:PinHeader_1x05_P2.54mm_Horizontal -> Connector_PinHeader_2.54mm:PinHeader_1x04_P2.54mm_Horizontal
- moved JP3 1.91 mm to (139.7, 78.7), turned to -90 degrees
- moved JP4 1.91 mm to (139.7, 73.7), turned to -90 degrees
- moved J13 1.27 mm to (144.8, 72.4)
- moved J14 1.27 mm to (158.8, 72.4)
Connections:
- net /LED_PWM renamed /A0/D0
- U2 pad 13: /1Wire -> /A10/D10
- U2 pad 3: /STATUS_LED -> /A1/D1
Routing:
- net /1Wire: track 40.0 -> 0.00 mm
- net /A10/D10: track 0.00 -> 32.4 mm
- net /STATUS_LED: track 13.2 -> 0.00 mm
- net /A1/D1: track 0.00 -> 13.2 mm
- net /SDO: track 15.1 -> 3.78 mm
- net +5V: track 92.4 -> 84.8 mm
- net /PS: track 17.8 -> 14.2 mm
- net +3V3: track 33.2 -> 36.5 mm
- net Net-(D6-A): track 1.80 -> 0.00 mm
- net (no net): track 0.00 -> 1.80 mm
- net /AD/CS: track 17.3 -> 16.3 mm
- net /SDA/SDI: track 16.8 -> 17.4 mm

Commit message: .
Parts:
- removed J1: Conn_Coaxial, Connector_Coaxial:BNC_TEConnectivity_1478204_Vertical
- removed M1: EZO-EC, KiCad Footprints:EZO_Conductivity_Module
- added C11: 100uF, Capacitor_SMD:C_0805_2012Metric_Pad1.18x1.45mm_HandSolder, F.Cu at (156.2, 97.5)
- added C12: 10uF, Capacitor_SMD:C_0805_2012Metric_Pad1.18x1.45mm_HandSolder, F.Cu at (156.2, 100.5)
- added C18: 10uF, Capacitor_SMD:C_0805_2012Metric_Pad1.18x1.45mm_HandSolder, F.Cu at (156.2, 103.5)
- added C19: 100nF, Capacitor_SMD:C_0805_2012Metric_Pad1.18x1.45mm_HandSolder, F.Cu at (156.2, 106.6)
- added C20: 100nF, Capacitor_SMD:C_0805_2012Metric_Pad1.18x1.45mm_HandSolder, F.Cu at (156.2, 109.6)
- added U4: TPS60400DBV, Package_TO_SOT_SMD:SOT-23-5, F.Cu at (161.2, 98.4)
- J13, J14: value Head Connector -> Pressure Transducer
Connections:
- net /AD/CS renamed /Pressure Transducer/AD/CS
- net /PS renamed /Pressure Transducer/PS
- net /SDO renamed /Pressure Transducer/SDO
- J13 pad 3: /SCL/SCLK -> /Pressure Transducer/SCL/SCLK
- J13 pad 4: /SDA/SDI -> /Pressure Transducer/SDA/SDI
- J15 pad 3: /SDA/SDI -> /Pressure Transducer/SDA/SDI
- J15 pad 4: /SCL/SCLK -> /Pressure Transducer/SCL/SCLK
- M2 pad 1: /SCL/SCLK -> /Pressure Transducer/SCL/SCLK
- M2 pad 7: /SDA/SDI -> /Pressure Transducer/SDA/SDI
- R14 pad 2: /SDA/SDI -> /Pressure Transducer/SDA/SDI
- R15 pad 2: /SCL/SCLK -> /Pressure Transducer/SCL/SCLK
Routing:
- net (no net): track 1.80 -> 43.6 mm
- net /A10/D10: track 32.4 -> 4.27 mm
- net Net-(J1-Ext): track 27.6 -> 0.00 mm
- net /SDA/SDI: track 17.4 -> 0.00 mm, vias 1 -> 0
- net /Pressure Transducer/SDA/SDI: track 0.00 -> 17.4 mm, vias 0 -> 1
- net /SCL/SCLK: track 15.5 -> 0.00 mm, vias 1 -> 0
- net /Pressure Transducer/SCL/SCLK: track 0.00 -> 15.5 mm, vias 0 -> 1
- net Net-(J1-In): track 14.3 -> 0.00 mm
- net +5V: track 84.8 -> 79.2 mm
