File: KiCAD/ROV CTD.kicad_sch (KiCad schematic)
At the start: 52 parts, among them J4 Bottom - Middle, J6 Main In, J7 Bottom - Middle, J8 Middle - Top, J9 Middle - Top, U1 AL8805W5, U2 ATtiny1614-Arduino, U3 AP63205WU, U6 MAX3072E

Commit message: cleanup
Parts:
- removed C10, C11, C12, C18: 47uF, Capacitor_SMD:C_0805_2012Metric_Pad1.18x1.45mm_HandSolder, symbol Device:C_Small
- removed C2: 2.2uF, Capacitor_SMD:C_0805_2012Metric_Pad1.18x1.45mm_HandSolder, symbol Device:C_Small
- removed C5: 1uF, Capacitor_SMD:C_0805_2012Metric_Pad1.18x1.45mm_HandSolder, symbol Device:C_Small
- removed C8: 100nF, Capacitor_SMD:C_0805_2012Metric_Pad1.18x1.45mm_HandSolder, symbol Device:C_Small
- removed D1: CXA1304, KiCad Footprints:LED - CXA1304, symbol Device:LED_Small_Filled
- removed D11: Status, LED_SMD:LED_0805_2012Metric_Pad1.15x1.40mm_HandSolder, symbol Device:LED_Small_Filled
- removed D2: BAT54S, Package_TO_SOT_SMD:SOT-23, symbol KiCad Symbols:BAT54S
- removed D6, D7, D8, D9: Inolux_IN-PI554FCH, LED_SMD:LED_Inolux_IN-PI554FCH_PLCC4_5.0x5.0mm_P3.2mm, symbol LED:Inolux_IN-PI554FCH
- removed J9: Middle - Top, Connector_PinHeader_1.27mm:PinHeader_2x03_P1.27mm_Vertical_SMD, symbol Connector_Generic:Conn_02x03_Odd_Even
- removed L1: SRN6045-330M, KiCad Footprints:inductor_33uH, symbol Partsbox:SRN6045-330M
- removed R1, R2, R5, R6: 0.5, Resistor_SMD:R_1206_3216Metric_Pad1.30x1.75mm_HandSolder, symbol Device:R_Small
- removed R12, R13: 330, Resistor_SMD:R_0805_2012Metric_Pad1.20x1.40mm_HandSolder, symbol Device:R_Small
- removed R14: 1k, Resistor_SMD:R_0805_2012Metric_Pad1.20x1.40mm_HandSolder, symbol Device:R_Small
- removed R3, R8: 10k, Resistor_SMD:R_0805_2012Metric_Pad1.20x1.40mm_HandSolder, symbol Device:R_Small
- removed TH1: NTCG203NH103JTDS, Resistor_SMD:R_0805_2012Metric_Pad1.20x1.40mm_HandSolder, symbol Partsbox:NTCG203NH103JTDS
- removed U1: AL8805W5, TO_SOT_Packages_SMD:SOT-23-5, symbol Partsbox:AL8860WT-7
Connections:
- net LED+_L: no longer names the net of J8.6 (Pin_6)
- net LED-_L: no longer names the net of J8.4 (Pin_4)
- net Neo_Mid: no longer names the net of J8.3 (Pin_3)
- net Neo_Mid: no longer J7.6 (Pin_6)
- net PWM: no longer names the net of J7.9 (Pin_9)
- net STATUS: no longer names the net of J8.5 (Pin_5)
- net STATUS: no longer J7.11 (Pin_11)
- no-connect marks 4 -> 3
Other:
- note removed: "400 mA current limit"
- title: ROV Light Module -> ROV CTD

Commit message: .
Parts:
- added C10: 47uF, Capacitor_SMD:C_0805_2012Metric_Pad1.18x1.45mm_HandSolder, symbol Device:C_Small
- added C5: 100nF, Capacitor_SMD:C_0805_2012Metric_Pad1.18x1.45mm_HandSolder, symbol Device:C_Small
- added C6: 10pF, Capacitor_SMD:C_0805_2012Metric_Pad1.18x1.45mm_HandSolder, symbol Device:C_Small
- added J10: 1Wire1, Connector_PinHeader_2.54mm:PinHeader_1x03_P2.54mm_Vertical, symbol Connector:Conn_01x03_Pin
- added J11: 1Wire2, Connector_PinHeader_2.54mm:PinHeader_1x03_P2.54mm_Vertical, symbol Connector:Conn_01x03_Pin
- added J12: 1Wire3, Connector_PinHeader_2.54mm:PinHeader_1x03_P2.54mm_Vertical, symbol Connector:Conn_01x03_Pin
- added J9: Middle - Top, Connector_PinHeader_1.27mm:PinHeader_2x03_P1.27mm_Vertical_SMD, symbol Connector_Generic:Conn_02x03_Odd_Even
Connections:
- net +5V_Mid: now also C10.1, C5.1, C6.1, J10.1 (Pin_1), J11.1 (Pin_1), J12.1 (Pin_1); no longer J8.2 (Pin_2)
- net GND: now also C10.2, C5.2, C6.2, J10.3 (Pin_3), J11.3 (Pin_3), J12.3 (Pin_3); no longer J8.1 (Pin_1)
- net 1Wire: now reaches J7.6 (Pin_6)
- net 1Wire: now also J10.2 (Pin_2), J11.2 (Pin_2), J12.2 (Pin_2)
Other:
- moved on the sheet: J8

Commit message: .
Parts:
- added J13: Conn_01x04_Pin, Connector_PinHeader_2.54mm:PinHeader_1x04_P2.54mm_Vertical, symbol Connector:Conn_01x04_Pin
- J7: value Bottom - Middle -> Middle - Bottom
- J9: value Middle - Top -> Top - Middle
Changed lines of the file:
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@@
+	)
+	(symbol
+		(lib_id "Connector:Conn_01x04_Pin")
+		(at 163.83 106.68 0)
+		(mirror y)
+		(unit 1)
+		(body_style 1)
+		(exclude_from_sim no)
+		(in_bom yes)
+		(on_board yes)
+		(in_pos_files yes)
+		(dnp no)
+		(fields_autoplaced yes)
+		(property "Reference" "J13"
+			(at 165.1 106.6799 0)
+			(show_name no)
+			(do_not_autoplace no)
+			(effects
+				(font
+					(size 1.27 1.27)
+				)
+				(justify right)
+			)
+		)
+		(property "Value" "Conn_01x04_Pin"
+			(at 165.1 109.2199 0)
+			(show_name no)
+			(do_not_autoplace no)
+			(effects
+				(font
+					(size 1.27 1.27)
+				)
+				(justify right)
+			)
+		)
+		(property "Footprint" "Connector_PinHeader_2.54mm:PinHeader_1x04_P2.54mm_Vertical"
+			(at 163.83 106.68 0)
+			(hide yes)
+			(show_name no)
+			(do_not_autoplace no)
+			(effects
+				(font
+					(size 1.27 1.27)
+				)
+			)
+		)
+		(property "Datasheet" ""
+			(at 163.83 106.68 0)
+			(hide yes)
+			(show_name no)
+			(do_not_autoplace no)
+			(effects
+				(font
+					(size 1.27 1.27)
+				)
+			)
+		)
+		(property "Description" "Generic connector, single row, 01x04, script generated"
+			(at 163.83 106.68 0)
+			(hide yes)
+			(show_name no)
+			(do_not_autoplace no)
+			(effects
+				(font
+					(size 1.27 1.27)
+				)
+			)
+		)
+		(pin "3"
+		)
+		(pin "1"
+		)
+		(pin "2"
+		)
+		(pin "4"
+		)
+		(instances
+			(project "ROV CTD"
+				(path "/4b85b8a1-3b52-4af9-b3a4-471ab529b035"
+					(reference "J13")
+					(unit 1)
+				)
+			)
+		)
 	)
 	(symbol
@@
 			)
 		)
-		(property "Value" "Middle - Top"
+		(property "Value" "Top - Middle"
 			(at 236.22 157.48 0)
 			(show_name no)
@@
 			)
 		)
-		(property "Value" "Bottom - Middle"
+		(property "Value" "Middle - Bottom"
 			(at 68.58 111.76 0)
 			(show_name no)
