File: KiCAD/ROV CTD.kicad_sch (KiCad schematic)
At the start: 34 parts, among them J10 1Wire1, J11 1Wire2, J12 1Wire3, J13 Conn_01x04_Pin, J4 Bottom - Middle, J6 Main In, J7 Middle - Bottom, J8 Middle - Top, J9 Top - Middle, U1 EZO-EC, U2 ATtiny1614-Arduino, U3 AP63205WU, U6 MAX3072E

Commit message: .
Parts:
- removed J13: Conn_01x04_Pin, Connector_PinHeader_2.54mm:PinHeader_1x04_P2.54mm_Vertical, symbol Connector:Conn_01x04_Pin
- removed J4: Bottom - Middle, Connector_PinSocket_1.27mm:PinSocket_2x06_P1.27mm_Vertical_SMD, symbol Connector_Generic:Conn_02x06_Odd_Even
- removed J7: Middle - Bottom, Connector_PinHeader_1.27mm:PinHeader_2x06_P1.27mm_Vertical_SMD, symbol Connector_Generic:Conn_02x06_Odd_Even
- removed J8: Middle - Top, Connector_PinSocket_1.27mm:PinSocket_2x03_P1.27mm_Vertical_SMD, symbol Connector_Generic:Conn_02x03_Odd_Even
- removed J9: Top - Middle, Connector_PinHeader_1.27mm:PinHeader_2x03_P1.27mm_Vertical_SMD, symbol Connector_Generic:Conn_02x03_Odd_Even
- added J1: Conn_Coaxial, Connector_Coaxial:BNC_TEConnectivity_1478204_Vertical, symbol Connector:Conn_Coaxial
- added J13: Interface, Connector_PinSocket_2.54mm:PinSocket_1x05_P2.54mm_Vertical, symbol Connector:Conn_01x05_Pin
- added J14: Interface, Connector_PinHeader_2.54mm:PinHeader_1x05_P2.54mm_Horizontal, symbol Connector:Conn_01x05_Pin
- renumbered U1 to M1
Connections:
- net +5V_Mid is gone; now on net +5V: C10.1, C5.1, C6.1, J10.1 (Pin_1), J11.1 (Pin_1), J12.1 (Pin_1), M1.4 (VCC)
- net NeoPixle is gone; now on net 1Wire: U2.13 (~A10/D10_SCK)
- net at M1.5 (PRB-Core): now also J1.1 (In)
- net at M1.6 (PRB-Sheild): now also J1.2 (Ext)
- no-connect marks 3 -> 0
Other:
- moved on the sheet: M1

Commit message: .
Parts:
- added D6: Status, LED_SMD:LED_0805_2012Metric_Pad1.15x1.40mm_HandSolder, symbol Device:LED_Small_Filled
- added J15: Conn_01x07_Pin, Connector_PinSocket_2.54mm:PinSocket_1x07_P2.54mm_Vertical, symbol Connector:Conn_01x07_Pin
- added R8: 520, Resistor_SMD:R_0805_2012Metric_Pad1.20x1.40mm_HandSolder, symbol Device:R_Small
Connections:
- net GND: now also D6.1 (K), J15.1 (Pin_1)
- net STATUS_LED: now also R8.1
- new net: D6.2 (A), R8.2
Other:
- moved on the sheet: J13

Commit message: .
Parts:
- added C7: 100nF, Capacitor_SMD:C_0805_2012Metric_Pad1.18x1.45mm_HandSolder, symbol Device:C_Small
- added JP3, JP4: RX, Jumper:SolderJumper-2_P1.3mm_Open_TrianglePad1.0x1.5mm, symbol Jumper:SolderJumper_2_Open
- added M2: MS5803-14BA, KiCad Footprints:MS5803-14BA, symbol KiCad Symbols:MS5803-14BA
- added R12, R13: 10k, Resistor_SMD:R_0805_2012Metric_Pad1.20x1.40mm_HandSolder, symbol Device:R_Small
- added R14, R15: 2k2, Resistor_SMD:R_0805_2012Metric_Pad1.20x1.40mm_HandSolder, symbol Device:R_Small
Connections:
- net GND: now also J13.1 (Pin_1), J14.1 (Pin_1), C7.2, JP3.1 (A), JP4.1 (A), M2.2 (GND)
- net +3V3: now reaches J13.2 (Pin_2)
- net +3V3: now also J14.2 (Pin_2), J15.2 (Pin_2), C7.1, M2.5 (VDD), R12.1, R13.1, R14.1, R15.1
- net SDA/SDI: now reaches J15.3 (Pin_3)
- net SDA/SDI: now also M2.7 (SDI/SDA), R14.2
- net SCL/SCLK: now reaches J15.4 (Pin_4)
- net SCL/SCLK: now also M2.1 (SCLK), R15.2
- net SDO: now reaches J15.5 (Pin_5)
- net SDO: now also M2.8 (SDO)
- net AD/CS: now reaches J15.6 (Pin_6)
- net AD/CS: now also JP4.2 (B), M2.3 (CSB), R13.2
- net PS: now reaches J15.7 (Pin_7)
- net PS: now also JP3.2 (B), M2.6 (PS), R12.2
Other:
- note added: "I2C by defult, Default address 0x76"
- moved on the sheet: J15

Commit message: .
Parts:
- J15: now not fitted
Connections:
- net SCL/SCLK: now also J13.3 (Pin_3)
- net SDA/SDI: now also J13.4 (Pin_4)
- net SDO: now also J13.5 (Pin_5)
Other:
- moved on the sheet: J13
