File: KiCAD/ROV CTD.kicad_sch (KiCad schematic)
At the start: 43 parts, among them J1 Conn_Coaxial, J10 1Wire1, J11 1Wire2, J12 1Wire3, J13 Interface, J14 Interface, J15 Conn_01x07_Pin, J6 Main In, M1 EZO-EC, M2 MS5803-14BA, U2 ATtiny1614-Arduino, U3 AP63205WU, U6 MAX3072E

Commit message: .
Connections:
- net SCL/SCLK: now also J14.3 (Pin_3)
- net SDA/SDI: now also J14.4 (Pin_4)
- net SDO: now also J14.5 (Pin_5)
Other:
- note removed: "Middle Board"
- moved on the sheet: C13, C7, D10, D4, J10, J11, J12, J13, J14, J15, R10, R11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

Commit message: .
Parts:
- removed D6: Status, LED_SMD:LED_0805_2012Metric_Pad1.15x1.40mm_HandSolder, symbol Device:LED_Small_Filled
- removed J10: 1Wire1, Connector_PinHeader_2.54mm:PinHeader_1x03_P2.54mm_Vertical, symbol Connector:Conn_01x03_Pin
- removed J11: 1Wire2, Connector_PinHeader_2.54mm:PinHeader_1x03_P2.54mm_Vertical, symbol Connector:Conn_01x03_Pin
- removed J12: 1Wire3, Connector_PinHeader_2.54mm:PinHeader_1x03_P2.54mm_Vertical, symbol Connector:Conn_01x03_Pin
- removed R8: 520, Resistor_SMD:R_0805_2012Metric_Pad1.20x1.40mm_HandSolder, symbol Device:R_Small
- added C8: 100nF, Capacitor_SMD:C_0805_2012Metric_Pad1.18x1.45mm_HandSolder, symbol Device:C_Small
- added H1, H2: Through Hole, MountingHole:MountingHole_3mm, symbol Mechanical:MountingHole
- J13: value Interface -> Head Connector; footprint Connector_PinSocket_2.54mm:PinSocket_1x05_P2.54mm_Vertical -> Connector_PinSocket_2.54mm:PinSocket_1x04_P2.54mm_Vertical; symbol Connector:Conn_01x05_Pin -> Connector:Conn_01x04_Socket
- J14: value Interface -> Head Connector; footprint Connector_PinHeader_2.54mm:PinHeader_1x05_P2.54mm_Horizontal -> Connector_PinHeader_2.54mm:PinHeader_1x04_P2.54mm_Horizontal; symbol Connector:Conn_01x05_Pin -> Connector:Conn_01x04_Pin
Connections:
- net +3V3: now also C8.1
- net GND: now also C8.2
- net SDO: no longer J13.5 (Pin_5), J14.5 (Pin_5)
- net 1Wire renamed A10/D10
- net LED_PWM renamed A0/D0
- net STATUS_LED renamed A1/D1
Other:
- moved on the sheet: J1, M1

Commit message: .
Parts:
- removed C7, C8: 100nF, Capacitor_SMD:C_0805_2012Metric_Pad1.18x1.45mm_HandSolder, symbol Device:C_Small
- removed J1: Conn_Coaxial, Connector_Coaxial:BNC_TEConnectivity_1478204_Vertical, symbol Connector:Conn_Coaxial
- removed J13: Head Connector, Connector_PinSocket_2.54mm:PinSocket_1x04_P2.54mm_Vertical, symbol Connector:Conn_01x04_Socket
- removed J15: Conn_01x07_Pin, Connector_PinSocket_2.54mm:PinSocket_1x07_P2.54mm_Vertical, symbol Connector:Conn_01x07_Pin
- removed JP3, JP4: RX, Jumper:SolderJumper-2_P1.3mm_Open_TrianglePad1.0x1.5mm, symbol Jumper:SolderJumper_2_Open
- removed M1: EZO-EC, KiCad Footprints:EZO_Conductivity_Module, symbol KiCad Symbols:EZO-EC
- removed M2: MS5803-14BA, KiCad Footprints:MS5803-14BA, symbol KiCad Symbols:MS5803-14BA
- removed R12, R13: 10k, Resistor_SMD:R_0805_2012Metric_Pad1.20x1.40mm_HandSolder, symbol Device:R_Small
- removed R14, R15: 2k2, Resistor_SMD:R_0805_2012Metric_Pad1.20x1.40mm_HandSolder, symbol Device:R_Small
- added D6: 3V3, LED_SMD:LED_0805_2012Metric_Pad1.15x1.40mm_HandSolder, symbol Device:LED_Small_Filled
- added D7: -3V3, LED_SMD:LED_0805_2012Metric_Pad1.15x1.40mm_HandSolder, symbol Device:LED_Small_Filled
- added R16, R8: 1k, Resistor_SMD:R_0805_2012Metric_Pad1.20x1.40mm_HandSolder, symbol Device:R_Small
- D10: value Power -> 5V
- J14: value Head Connector -> Pressure Transducer
- R11: value 470 -> 1k
Connections:
- net +3V3: now also R8.1
- net GND: now also D6.1 (K), D7.1 (K)
- new net: D7.2 (A), R16.2
- new net: D6.2 (A), R8.2
- new net -3V3: R16.1
Other:
- added sheet Conductivity Transducer (Conductivity Transducer.kicad_sch)
- added sheet Pressure Transducer (Pressure Transducer.kicad_sch)
- note removed: "I2C by defult, Default address 0x76"
- moved on the sheet: C10, C5, C6, D10, D4, R11, R7
